File: demo_carte_led/demo_carte_led.kicad_pcb (KiCad board)
At the start: 2 copper layers, 42 x 24 mm, 5 parts, among them J1 GROVE

Commit message: Mise à jour vers KiCAD 6 + Fichier FreeCAD
Connections:
- J1 pad 3: (no net) -> unconnected-(J1-Pad3)
Other:
- net class Default removed
